File: MQTT-Agent-Hardware/CPU PCB/ESP32c6 Agent PCB CPU.kicad_pcb (KiCad board)
At the start: 2 copper layers, 50.8 x 40 mm, 19 parts, among them J1 Screw_Terminal_01x14, J2 Power, SW1 SW_Push, SW2 SW_Push, SW3 SW_Push, U2 DFPlayer_Module, U5 XIAO-ESP32-C6, U6 74AHCT125

Commit message: Cleanup and Finalize.
Updated footprints.
cleaned up silkscreen.
Changed schematic to B-size
Parts:
- removed J2: Power, Connector_Molex:Molex_KK-254_AE-6410-02A_1x02_P2.54mm_Vertical
- added J10: Power, Connector_Molex:Molex_KK-254_AE-6410-02A_1x02_P2.54mm_Vertical, F.Cu at (143.2, 54.4)
- U1: footprint MDS_Library:SSD1306-128x32 -> MDS_Library:SSD1306-128x32_Borderless
Routing:
- net GND: track 214.0 -> 207.2 mm
- net Net-(U5-GPIO20/D9/MISO): track 37.4 -> 39.5 mm

Commit message: Cleanup
Parts:
- added JP1: GPIO16 Direct, Jumper:SolderJumper-2_P1.3mm_Open_Pad1.0x1.5mm, F.Cu at (130.2, 79.5)
- added JP2: GPIO17 Direct, Jumper:SolderJumper-2_P1.3mm_Open_Pad1.0x1.5mm, F.Cu at (137.8, 63.5)
- moved C4 2.50 mm to (111.0, 54.6)
- moved U2 0.30 mm to (134.0, 72.9)
Routing:
- net GND: track 207.2 -> 103.1 mm, vias 0 -> 15
- net DAC-L: track 30.0 -> 44.1 mm, vias 1 -> 2
- net /TX: track 13.4 -> 24.8 mm
- net Net-(JP2-A): track 16.8 -> 26.9 mm
- net /I.1: track 67.6 -> 59.3 mm
- net Net-(U1-SDA): track 45.9 -> 37.6 mm
- net /~{CFG}: track 41.4 -> 46.5 mm
- net DAC-R: track 30.3 -> 33.2 mm, vias 1 -> 2
- net /I.0: track 58.8 -> 56.4 mm
- net /T.0: track 61.5 -> 63.6 mm
- net VCC: track 100.3 -> 98.8 mm
- net /O5.0: track 21.8 -> 23.2 mm
- net /O5.1: track 26.4 -> 25.2 mm
- net +3V3: track 127.9 -> 127.0 mm
- net /O.1: track 56.5 -> 57.3 mm
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- added copper zone on B.Cu, net GND
Other:
- board text added: "(c) 2026 Marc D. Spencer"
- board text added: "MQTT Agent 5.0b"
- board text removed: "MQTT Agent 5.0b (c) 2026 Marc D. Spencer"
